File: pcb/MosaicE.kicad_pcb (KiCad board)
At the start: 2 copper layers, 61.6 x 40.4 mm, 13 parts, among them SW1 SW_Push, SW2 SW_Push, SW3 SW_Push, SW4 RotaryEncoder, U1 XIAO-RP2040-DIP

Commit message: src files added
Parts:
- added G***: LOGO, LOGO, B.Cu at (85.9, 106.0)
- added G***: LOGO, LOGO, B.Cu at (114.2, 105.9)
