File: pcb/MosaicE.kicad_sch (KiCad schematic)
At the start: 13 parts, among them SW1 SW_Push, SW2 SW_Push, SW3 SW_Push, SW4 RotaryEncoder, U1 XIAO-RP2040-DIP

Commit message: src files added
Other:
- moved on the sheet: D5, D6, D7, D8, R1, R2, R3, R4, SW4, U1
